File: Schematic_01.brd (EAGLE design)
At the start: 100 x 100 mm, 153 parts, among them Q1 32.768Khz, U1 STM32F103RET6, U2 STM32F103C8T6, U3 AMS1117-3.3, U4 AMS1117-3.3, U5 AZ1117-5.0, U6 AMS1117-3.3, U7 MBT3904DW1T1G, U8 BC846A, U9 FDV304P

Commit message: Added a "Somewhat" of an Main Board Layout + PDF and PNG :)
Parts:
- removed Q1: 32.768Khz, crystal:TC26H
- removed U$13: SMD_FERRITE_BEAD, STMBerry:0805
- removed U$21, U$3: ZTT8.00MT, STMBerry:ZTT8.00MT
- added C28, C29, C30, C31: 30pF, rcl:C0805K
- added FB: SMD_FERRITE_BEAD, STMBerry:0805
- added Q2, Q3: 8Mhz, crystal:SM49
- added Q4: 32.768Khz, crystal:MC-306
- C2, C3: value 20nF -> 20pF
- moved PH36 280.2 mm to (104.2, -84.8), turned to 270 degrees
- moved PH25 270.8 mm to (38.7, -71.7)
- moved C12 269.2 mm to (82.2, 10.3), flipped to the bottom, turned to 90 degrees
- moved PH26 260.6 mm to (83.3, -23.4), turned to 90 degrees
- moved C13 257.6 mm to (77.3, 10.7), flipped to the bottom, turned to 270 degrees
- moved PH12 256.0 mm to (72.7, -48.6)
- moved PH13 254.5 mm to (76.6, -42.6)
- moved PH38 252.0 mm to (106.4, -53.7), turned to 180 degrees
- moved PH39 247.1 mm to (118.5, -45.1), turned to 270 degrees
- moved PH37 225.2 mm to (64.8, -43.9), turned to 180 degrees
- moved C6 223.4 mm to (72.8, 23.1), flipped to the bottom, turned to 270 degrees
- moved C9 219.8 mm to (61.1, 23.1), flipped to the bottom, turned to 90 degrees
- moved C23 214.8 mm to (57.5, 23.1), flipped to the bottom, turned to 270 degrees
- moved C10 212.6 mm to (38.4, 42.7), turned to 270 degrees
- moved C11 206.7 mm to (34.4, 42.9), turned to 90 degrees
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Connections:
- net AGND: now also FB.P$4; no longer U$13.P$4
- net GND: now also C28.1, C29.2, C30.1, C31.2, FB.P$3; no longer U$13.P$3, U$21.2, U$3.2
- net N$4: now also C29.1, Q3.1; no longer U$21.3
- net N$45: now also C30.2, Q2.2; no longer U$3.1
- net N$46: now also C31.1, Q2.1; no longer U$3.3
- net N$6: now also Q4.4; no longer Q1.2
- net N$8: now also Q4.1; no longer Q1.1
- net N$9: now also C28.2, Q3.2; no longer U$21.1
Routing:
- net 3.3V: track 69.8 -> 0.00 mm, vias 4 -> 0
- net BMP_TXD: track 60.7 -> 0.00 mm, vias 2 -> 0
- net BMP_RXD: track 56.0 -> 0.00 mm, vias 2 -> 0
- net BMP_BUT: track 45.8 -> 0.00 mm, vias 3 -> 0
- net 5V: track 35.4 -> 0.00 mm, vias 1 -> 0
- net N$41: track 23.9 -> 0.00 mm, vias 2 -> 0
- net BMP_LED1: track 21.3 -> 0.00 mm, vias 3 -> 0
- net BMP_RST: track 20.9 -> 0.00 mm
- net BMP_LED0: track 18.8 -> 0.00 mm, vias 1 -> 0
- net BMP_LED2: track 17.8 -> 0.00 mm, vias 1 -> 0
- net N$50: track 17.7 -> 0.00 mm, vias 1 -> 0
- net BMP_TDI: track 17.5 -> 0.00 mm
- net BMP_DP: track 17.2 -> 0.00 mm, vias 2 -> 0
- net BMP_TDO: track 17.2 -> 0.00 mm, vias 1 -> 0
- net TPWR: track 15.9 -> 0.00 mm, vias 1 -> 0
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