File: Schematic_01.sch (EAGLE design)
At the start: 153 parts, among them Q1 32.768Khz, U1 STM32F103RET6, U2 STM32F103C8T6, U3 AMS1117-3.3, U4 AMS1117-3.3, U5 AZ1117-5.0, U6 AMS1117-3.3, U7 MBT3904DW1T1G, U8 BC846A, U9 FDV304P

Commit message: Added a "Somewhat" of an Main Board Layout + PDF and PNG :)
Parts:
- removed Q1: 32.768Khz, crystal:CRYTALTC26H
- removed U$21, U$3: ZTT8.00MT, STMBerry:ZTT8.00MT
- added C28, C29, C30, C31: 30pF, rcl:C-EUC0805K
- added Q2, Q3: 8Mhz, crystal:CRYSTALSM49
- added Q4: 32.768Khz, crystal:MC-306
- C2, C3: value 20nF -> 20pF
- renumbered U$13 to FB
Connections:
- net GND: now also C28.1, C29.2, C30.1, C31.2; no longer U$21.2, U$3.2
- net N$4: now also C29.1, Q3.1; no longer U$21.3
- net N$45: now also C30.2, Q2.2; no longer U$3.1
- net N$46: now also C31.1, Q2.1; no longer U$3.3
- net N$6: now also Q4.2; no longer Q1.2
- net N$8: now also Q4.1; no longer Q1.1
- net N$9: now also C28.2, Q3.2; no longer U$21.1
